File: pcb/power.kicad_sch (KiCad schematic)
At the start: 29 parts, among them J2 USB_B_Micro, J4 Battery, J5 Cradle, U10 MAX17048, U11 MCP73831, U3 USBLC6-2, U4 RT9080-3.3, U5 LM66200DRLR, U6 LM66200DRLR, U8 SPX3819M5-L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

Commit message: more schematic updates
Parts:
- added D35: P6SMB12CA, Diode_SMD:D_SMB, symbol Device:D_TVS
Connections:
- net +8V: now also D35.2 (A2)
- net GND: now also J4.3 (Pin_3), D35.1 (A1)
- net VBATT: now also J4.1 (Pin_1)
Other:
- note added: "1 2 3"
- moved on the sheet: J4, J5, R3

Commit message: cradle connector
Connections:
- net +8V: now also J5.1 (Pin_1); no longer J5.3 (Pin_3)
- net GND: now also J5.2 (Pin_2); no longer J5.1 (Pin_1)
- no-connect marks 1 -> 2
Other:
- note removed: "Confirm Cradel pinout"

Commit message: parts placed
Parts:
- C10, C11, C13, C14, C15, C16, C8, C9: footprint SparkFun-Capacitor:C_0402_1005Metric -> Capacitor_SMD:C_0805_2012Metric
- C12: footprint SparkFun-Capacitor:C_0603_1608Metric -> Capacitor_SMD:C_0805_2012Metric
- C5: value 10u -> .1u
- R11, R12: footprint (none) -> Resistor_SMD:R_0805_2012Metric
- U10: footprint SparkFun-Semiconductor-Standard:DFN-8 -> 880+:TDFN-8-1EP_2x2mm_P0.5mm_EP0.8x1.4mm
- U11, U4, U9: footprint SparkFun-Semiconductor-Standard:SOT23-5 -> Package_TO_SOT_SMD:SOT-23-5
- U5, U6: footprint SOT-5X3_DRL_TEX -> Package_TO_SOT_SMD:SOT-583-8
- renumbered D35 to TVS1
Connections:
- net +3.3VP: now also C5.1, C6.1
- net +5V: now also C12.1
- net +8V: now also F2.2; no longer J5.1 (Pin_1)
- net Cradel_input: now also R11.1, U8.5 (OUT); no longer F2.2
- net GND: now also C5.2, C6.2
- new net: F2.1, J5.1 (Pin_1)
Other:
- moved on the sheet: F2

Commit message: update todo and reference info
Other:
- note added: "Red Black White"
